Commit message: added SOMA-HOME Ontology for class extraction, changed to parse_urdf_SOMA, changed print in viz_marker

File: resources/apartment.urdf (robot description, URDF)
Before this commit: robot apartment, 117 links, 116 joints
Links:
- removed link coffe_machine
- added link coffee_machine; collision box size=0.58 0.32 0.41; visual box size=0.58 0.33 0.41
Joints:
- removed joint coffe_machine_joint
- added joint coffee_machine_joint: type fixed, parent countertop, child coffee_machine, origin xyz=0 0.3 0.2
